Commit message: added two Lidar frames to URDF. Lower and Upper.

File: ROS/omron_ld60_description/models/LD60_castors.urdf (robot description, URDF)
Before this commit: robot ld60_castors, 12 links, 11 joints
Links:
- added link lower_laser, mass 0.001
- added link upper_laser, mass 0.001
Joints:
- added joint main_body_to_lower_laser: type fixed, parent main_body, child lower_laser, origin xyz=0.27 0 -0.03
- added joint main_body_to_upper_laser: type fixed, parent main_body, child upper_laser, origin xyz=0.27 0 0.11
