Commit message: fixed TF bug

File: Unity/Omron_LD60/Assets/robot_model/LD60_castors.urdf (robot description, URDF)
Before this commit: robot ld60_castors, 14 links, 13 joints
Links:
- added link ignore_this_link
Joints:
- removed joint base_to_main_body
- added joint base_link_to_main_body: type fixed, parent base_link, child main_body, origin xyz=0 0 0.085
- added joint ignore_this_joint: type fixed, parent ignore_this_link, child base_link
